File: buzzybox/buzzybox.sch (KiCad schematic (older format))
At the start: 7 parts, among them J1 AudioJack2, J2 Barrel_Jack

Commit message: complete mini layout
Parts:
- removed J1: AudioJack2, Connectors:Stereo_Jack_3.5mm_Switch_Ledino_KB3SPRS, symbol Connector:AudioJack2
- added J1: AudioJack3, buzzybox:STX-3000, symbol Connector:AudioJack3
- added J3, J4: Conn_01x03, Connector_PinHeader_2.54mm:PinHeader_1x03_P2.54mm_Horizontal, symbol Connector_Generic:Conn_01x03
- H1: footprint (none) -> MountingHole:MountingHole_3.2mm_M3_Pad
- H2, H3, H4: renamed from H?; footprint (none) -> MountingHole:MountingHole_3.2mm_M3_Pad
- renumbered C1 to C11
Connections:
- net +VDC: now also J3.1 (Pin_1), J4.1 (Pin_1)
- net -VDC: now also J1.S, J3.2 (Pin_2), J4.2 (Pin_2)
- net at C11.2: now also J1.T, J3.3 (Pin_3), J4.3 (Pin_3)
- no-connect marks 0 -> 1
Changed lines of the file:
@@
 	1    0    0    -1
-$EndComp
-$Comp
-L Connector:AudioJack2 J1
-U 1 1 5FD4629F
-P 7200 3500
-F 0 "J1" H 7020 3483 50  0000 R CNN
-F 1 "AudioJack2" H 7020 3574 50  0000 R CNN
-F 2 "Connectors:Stereo_Jack_3.5mm_Switch_Ledino_KB3SPRS" H 7200 3500 50  0001 C CNN
-F 3 "~" H 7200 3500 50  0001 C CNN
-	1    7200 3500
-	-1   0    0    1
 $EndComp
 Wire Wire Line
@@
 L power:-VDC #PWR0103
 U 1 1 5FD495C3
-P 7000 3700
-F 0 "#PWR0103" H 7000 3600 50  0001 C CNN
-F 1 "-VDC" H 7000 3975 50  0000 C CNN
-F 2 "" H 7000 3700 50  0001 C CNN
-F 3 "" H 7000 3700 50  0001 C CNN
-	1    7000 3700
-	-1   0    0    1
-$EndComp
-Wire Wire Line
-	7000 3600 7000 3700
+P 7000 3800
+F 0 "#PWR0103" H 7000 3700 50  0001 C CNN
+F 1 "-VDC" H 7000 4075 50  0000 C CNN
+F 2 "" H 7000 3800 50  0001 C CNN
+F 3 "" H 7000 3800 50  0001 C CNN
+	1    7000 3800
+	-1   0    0    1
+$EndComp
+Wire Wire Line
+	7000 3700 7000 3800
 Wire Wire Line
 	2500 4000 3000 4000
@@
 Connection ~ 5500 4000
 $Comp
-L Device:C C1
+L Device:C C11
 U 1 1 5FD53811
 P 6250 3500
-F 0 "C1" V 6502 3500 50  0000 C CNN
+F 0 "C11" V 6502 3500 50  0000 C CNN
 F 1 "0.1uF" V 6411 3500 50  0000 C CNN
 F 2 "Capacitors_THT:C_Disc_D3.0mm_W1.6mm_P2.50mm" H 6288 3350 50  0001 C CNN
@@
 Connection ~ 5500 3500
 Wire Wire Line
-	6400 3500 7000 3500
+	6400 3500 6700 3500
 $Comp
 L Mechanical:MountingHole_Pad H1
@@
 F 0 "H1" H 5600 1449 50  0000 L CNN
 F 1 "M3" H 5600 1358 50  0000 L CNN
-F 2 "" H 5500 1400 50  0001 C CNN
+F 2 "MountingHole:MountingHole_3.2mm_M3_Pad" H 5500 1400 50  0001 C CNN
 F 3 "~" H 5500 1400 50  0001 C CNN
 	1    5500 1400
@@
 $EndComp
 $Comp
-L power:-VDC #PWR?
+L power:-VDC #PWR01
 U 1 1 5FD723DB
 P 6250 1650
-F 0 "#PWR?" H 6250 1550 50  0001 C CNN
+F 0 "#PWR01" H 6250 1550 50  0001 C CNN
 F 1 "-VDC" H 6250 1925 50  0000 C CNN
 F 2 "" H 6250 1650 50  0001 C CNN
@@
 $EndComp
 $Comp
-L Mechanical:MountingHole_Pad H?
+L Mechanical:MountingHole_Pad H2
 U 1 1 5FD733CC
 P 6000 1400
-F 0 "H?" H 6100 1449 50  0000 L CNN
+F 0 "H2" H 6100 1449 50  0000 L CNN
 F 1 "M3" H 6100 1358 50  0000 L CNN
-F 2 "" H 6000 1400 50  0001 C CNN
+F 2 "MountingHole:MountingHole_3.2mm_M3_Pad" H 6000 1400 50  0001 C CNN
 F 3 "~" H 6000 1400 50  0001 C CNN
 	1    6000 1400
@@
 $EndComp
 $Comp
-L Mechanical:MountingHole_Pad H?
+L Mechanical:MountingHole_Pad H3
 U 1 1 5FD73798
 P 6500 1400
-F 0 "H?" H 6600 1449 50  0000 L CNN
+F 0 "H3" H 6600 1449 50  0000 L CNN
 F 1 "M3" H 6600 1358 50  0000 L CNN
-F 2 "" H 6500 1400 50  0001 C CNN
+F 2 "MountingHole:MountingHole_3.2mm_M3_Pad" H 6500 1400 50  0001 C CNN
 F 3 "~" H 6500 1400 50  0001 C CNN
 	1    6500 1400
@@
 $EndComp
 $Comp
-L Mechanical:MountingHole_Pad H?
+L Mechanical:MountingHole_Pad H4
 U 1 1 5FD74397
 P 7000 1400
-F 0 "H?" H 7100 1449 50  0000 L CNN
+F 0 "H4" H 7100 1449 50  0000 L CNN
 F 1 "M3" H 7100 1358 50  0000 L CNN
-F 2 "" H 7000 1400 50  0001 C CNN
+F 2 "MountingHole:MountingHole_3.2mm_M3_Pad" H 7000 1400 50  0001 C CNN
 F 3 "~" H 7000 1400 50  0001 C CNN
 	1    7000 1400
@@
 Wire Wire Line
 	6250 1500 6500 1500
+$Comp
+L Connector:AudioJack3 J1
+U 1 1 5FD96D5A
+P 7200 3600
+F 0 "J1" H 6920 3533 50  0000 R CNN
+F 1 "AudioJack3" H 6920 3624 50  0000 R CNN
+F 2 "buzzybox:STX-3000" H 7200 3600 50  0001 C CNN
+F 3 "~" H 7200 3600 50  0001 C CNN
+	1    7200 3600
+	-1   0    0    1
+$EndComp
+NoConn ~ 7000 3600
+$Comp
+L Connector_Generic:Conn_01x03 J3
+U 1 1 5FDA9972
+P 7200 4600
+F 0 "J3" H 7280 4642 50  0000 L CNN
+F 1 "Conn_01x03" H 7280 4551 50  0000 L CNN
+F 2 "Connector_PinHeader_2.54mm:PinHeader_1x03_P2.54mm_Horizontal" H 7200 4600 50  0001 C CNN
+F 3 "~" H 7200 4600 50  0001 C CNN
+	1    7200 4600
+	1    0    0    -1
+$EndComp
+$Comp
+L Connector_Generic:Conn_01x03 J4
+U 1 1 5FDAA94A
+P 7200 5100
+F 0 "J4" H 7280 5142 50  0000 L CNN
+F 1 "Conn_01x03" H 7280 5051 50  0000 L CNN
+F 2 "Connector_PinHeader_2.54mm:PinHeader_1x03_P2.54mm_Horizontal" H 7200 5100 50  0001 C CNN
+F 3 "~" H 7200 5100 50  0001 C CNN
+	1    7200 5100
+	1    0    0    -1
+$EndComp
+$Comp
+L power:-VDC #PWR0124
+U 1 1 5FDAB422
+P 6250 4600
+F 0 "#PWR0124" H 6250 4500 50  0001 C CNN
+F 1 "-VDC" H 6250 4875 50  0000 C CNN
+F 2 "" H 6250 4600 50  0001 C CNN
+F 3 "" H 6250 4600 50  0001 C CNN
+	1    6250 4600
+	-1   0    0    1
+$EndComp
+$Comp
+L power:+VDC #PWR0125
+U 1 1 5FDAB8F4
+P 6250 4500
+F 0 "#PWR0125" H 6250 4400 50  0001 C CNN
+F 1 "+VDC" H 6250 4775 50  0000 C CNN
+F 2 "" H 6250 4500 50  0001 C CNN
+F 3 "" H 6250 4500 50  0001 C CNN
+	1    6250 4500
+	1    0    0    -1
+$EndComp
+Wire Wire Line
+	6250 4500 6500 4500
+Wire Wire Line
+	6250 4600 6600 4600
+Wire Wire Line
+	6500 4500 6500 5000
+Wire Wire Line
+	6500 5000 7000 5000
+Connection ~ 6500 4500
+Wire Wire Line
+	6500 4500 7000 4500
+Wire Wire Line
+	6600 4600 6600 5100
+Wire Wire Line
+	6600 5100 7000 5100
+Connection ~ 6600 4600
+Wire Wire Line
+	6600 4600 7000 4600
+Wire Wire Line
+	7000 5200 6700 5200
+Wire Wire Line
+	6700 5200 6700 4700
+Connection ~ 6700 3500
+Wire Wire Line
+	6700 3500 7000 3500
+Wire Wire Line
+	7000 4700 6700 4700
+Connection ~ 6700 4700
+Wire Wire Line
+	6700 4700 6700 3500
 $EndSCHEMATC

Commit message: finalize main PCB after parts recieved
Connections:
- net -VDC renamed GND
Changed lines of the file:
@@
 $EndSheet
-$Comp
-L power:-VDC #PWR0101
-U 1 1 5FD44C8B
-P 8750 2700
-F 0 "#PWR0101" H 8750 2600 50  0001 C CNN
-F 1 "-VDC" H 8750 2975 50  0000 C CNN
-F 2 "" H 8750 2700 50  0001 C CNN
-F 3 "" H 8750 2700 50  0001 C CNN
-	1    8750 2700
-	-1   0    0    1
-$EndComp
 $Comp
 L power:+VDC #PWR0102
@@
 Wire Wire Line
 	8500 2700 8750 2700
-$Comp
-L power:-VDC #PWR0103
-U 1 1 5FD495C3
-P 7000 3800
-F 0 "#PWR0103" H 7000 3700 50  0001 C CNN
-F 1 "-VDC" H 7000 4075 50  0000 C CNN
-F 2 "" H 7000 3800 50  0001 C CNN
-F 3 "" H 7000 3800 50  0001 C CNN
-	1    7000 3800
-	-1   0    0    1
-$EndComp
 Wire Wire Line
 	7000 3700 7000 3800
@@
 $EndComp
 $Comp
-L power:-VDC #PWR01
-U 1 1 5FD723DB
-P 6250 1650
-F 0 "#PWR01" H 6250 1550 50  0001 C CNN
-F 1 "-VDC" H 6250 1925 50  0000 C CNN
-F 2 "" H 6250 1650 50  0001 C CNN
-F 3 "" H 6250 1650 50  0001 C CNN
-	1    6250 1650
-	-1   0    0    1
-$EndComp
-$Comp
 L Mechanical:MountingHole_Pad H2
 U 1 1 5FD733CC
@@
 $EndComp
 $Comp
-L power:-VDC #PWR0124
-U 1 1 5FDAB422
-P 6250 4600
-F 0 "#PWR0124" H 6250 4500 50  0001 C CNN
-F 1 "-VDC" H 6250 4875 50  0000 C CNN
-F 2 "" H 6250 4600 50  0001 C CNN
-F 3 "" H 6250 4600 50  0001 C CNN
-	1    6250 4600
-	-1   0    0    1
-$EndComp
-$Comp
 L power:+VDC #PWR0125
 U 1 1 5FDAB8F4
@@
 Wire Wire Line
 	6700 4700 6700 3500
+$Comp
+L power:GND #PWR0101
+U 1 1 5FDA7A4C
+P 8750 2700
+F 0 "#PWR0101" H 8750 2450 50  0001 C CNN
+F 1 "GND" H 8755 2527 50  0000 C CNN
+F 2 "" H 8750 2700 50  0001 C CNN
+F 3 "" H 8750 2700 50  0001 C CNN
+	1    8750 2700
+	1    0    0    -1
+$EndComp
+$Comp
+L power:GND #PWR0103
+U 1 1 5FDA8214
+P 7000 3800
+F 0 "#PWR0103" H 7000 3550 50  0001 C CNN
+F 1 "GND" H 7005 3627 50  0000 C CNN
+F 2 "" H 7000 3800 50  0001 C CNN
+F 3 "" H 7000 3800 50  0001 C CNN
+	1    7000 3800
+	1    0    0    -1
+$EndComp
+$Comp
+L power:GND #PWR0105
+U 1 1 5FDA872D
+P 6250 4600
+F 0 "#PWR0105" H 6250 4350 50  0001 C CNN
+F 1 "GND" H 6255 4427 50  0000 C CNN
+F 2 "" H 6250 4600 50  0001 C CNN
+F 3 "" H 6250 4600 50  0001 C CNN
+	1    6250 4600
+	1    0    0    -1
+$EndComp
+$Comp
+L power:GND #PWR0107
+U 1 1 5FDA8B2F
+P 6250 1650
+F 0 "#PWR0107" H 6250 1400 50  0001 C CNN
+F 1 "GND" H 6255 1477 50  0000 C CNN
+F 2 "" H 6250 1650 50  0001 C CNN
+F 3 "" H 6250 1650 50  0001 C CNN
+	1    6250 1650
+	1    0    0    -1
+$EndComp
 $EndSCHEMATC
